Commit message: PiPER-X model, torque-mode drag/impedance examples, friction identification
The arm is a PiPER-X, not a PiPER: its firmware FK matches the piper_x URDF
to 0.01 mm (the piper model left 7.8 mm and a week of wrist ghosts - J4's
phantom ~1 N.m is just piper_x's off-axis link4 COM, J5's lever is 13 mm not
61 mm, J4/J5 limits are +/-89 deg). piper_description.urdf is now piper_x +
gripper merged from agilexrobotics/agx_arm_urdf@main.

Examples reorganized around torque control (piperx-teleop >= 0.2.0):
- drag_mode / impedance_demo: canonical consumers of the package's
  GravityCompensator and JointImpedance
- friction_id: per-joint M/f0/b + breakaway identification by trajectory
  regression under known MIT torques (the command is the label)
- balanced_drag, equal_power_drag, virtual_dynamics, virtual_joint: the
  friction/inertia balancing + virtual work (dW = F dx, F = k*I) research
  line, culminating in the two-regime stiction-matched virtual joint
- record_drag / replay_drag / leader_drag / drag_teach: firmware drag-mode
  (0xFA / MotionCtrl_1) recording and replay
- assert_arm_config, probe_teach_mode: firmware gravity-settings tools

config/admittance.toml + per-joint admittance tuning kept as the legacy
position-mode path (superseded by torque mode for the leader arm).

Co-Authored-By: Claude Fable 5 <noreply@anthropic.com>

File: piper_ht/piper_description.urdf (robot description, URDF)
Before this commit: robot piper, 11 links, 10 joints
Links:
- removed link dummy_link
- removed link link7
- removed link link8
- added link flange_link, mass 0.04; collision mesh filename=package://agx_arm_description/agx_arm_urdf/piper_x/meshes/f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; visual mesh filename=package://agx_arm_description/agx_arm_urdf/piper_x/meshes/d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
- added link gripper_link
- added link gripper_link1, mass 0.025; collision mesh filename=package://agx_arm_description/agx_arm_urdf/piper_x/meshes/g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; visual mesh filename=package://agx_arm_description/agx_arm_urdf/piper_x/meshes/d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
- added link gripper_link2, mass 0.025; collision mesh filename=package://agx_arm_description/agx_arm_urdf/piper_x/meshes/g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; visual mesh filename=package://agx_arm_description/agx_arm_urdf/piper_x/meshes/d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
- added link world
- link base_link: geometry collision mesh filename=package://agx_arm_description/agx_arm_urdf/piper_x/meshes/b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; visual mesh filename=package://agx_arm_description/agx_arm_urdf/piper_x/meshes/d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
- link gripper_base: geometry collision mesh filename=package://agx_arm_description/agx_arm_urdf/piper_x/meshes/g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; visual mesh filename=package://agx_arm_description/agx_arm_urdf/piper_x/meshes/d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
- link link1: geometry collision mesh filename=package://agx_arm_description/agx_arm_urdf/piper_x/meshes/l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; visual mesh filename=package://agx_arm_description/agx_arm_urdf/piper_x/meshes/d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
- link link2: mass 1.17 -> 1.16; geometry collision mesh filename=package://agx_arm_description/agx_arm_urdf/piper_x/meshes/l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; visual mesh filename=package://agx_arm_description/agx_arm_urdf/piper_x/meshes/d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
- link link3: mass 0.5 -> 0.67; geometry collision mesh filename=package://agx_arm_description/agx_arm_urdf/piper_x/meshes/l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; visual mesh filename=package://agx_arm_description/agx_arm_urdf/piper_x/meshes/d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
- link link4: mass 0.38 -> 0.39; geometry collision mesh filename=package://agx_arm_description/agx_arm_urdf/piper_x/meshes/l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; visual mesh filename=package://agx_arm_description/agx_arm_urdf/piper_x/meshes/d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
- link link5: mass 0.383 -> 0.35; geometry collision mesh filename=package://agx_arm_description/agx_arm_urdf/piper_x/meshes/l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; visual mesh filename=package://agx_arm_description/agx_arm_urdf/piper_x/meshes/d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
- link link6: geometry collision mesh filename=package://agx_arm_description/agx_arm_urdf/piper_x/meshes/l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; visual mesh filename=package://agx_arm_description/agx_arm_urdf/piper_x/meshes/d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
Joints:
- removed joint base_to_dummy
- removed joint joint6_to_gripper_base
- removed joint joint7
- removed joint joint8
- added joint flange_joint: type fixed, parent link6, child flange_link, origin xyz=0 0 0 rpy=0 0 0
- added joint gripper: type prismatic, parent gripper_base, child gripper_link, origin xyz=0 0 0 rpy=0 0 0, axis 0 0 1, limit lower=0 upper=0.1 effort=10 velocity=3
- added joint gripper_base_joint: type fixed, parent flange_link, child gripper_base, origin xyz=0 0 0.0045 rpy=0 0 1.5707963
- added joint gripper_joint1: type prismatic, parent gripper_base, child gripper_link1, origin xyz=0 0 0.138 rpy=1.5707963 0 0, axis 0 0 1, limit lower=0 upper=0.05 effort=10 velocity=3, mimic joint=gripper multiplier=0.5 offset=0.0
- added joint gripper_joint2: type prismatic, parent gripper_base, child gripper_link2, origin xyz=0 0 0.138 rpy=1.5707963 0 -3.1415926, axis 0 0 -1, limit lower=-0.05 upper=0 effort=10 velocity=3, mimic joint=gripper multiplier=-0.5 offset=0.0
- added joint world_to_base_link: type fixed, parent world, child base_link, origin xyz=0 0 0 rpy=0 0 0
- joint joint1: limit lower=-2.618 upper=2.618 effort=100 velocity=5 -> lower=-2.6179938 upper=2.6179938 effort=100 velocity=5; origin xyz=0 0 0.123 rpy=0 0 0 -> xyz=0 0 0.123 rpy=0 0 3.1415926
- joint joint2: limit lower=0 upper=3.14 effort=100 velocity=5 -> lower=0 upper=3.1415926 effort=100 velocity=5; origin xyz=0 0 0 rpy=1.5708 -0.1359 -3.1416 -> xyz=0 0 0 rpy=-1.5707963 -3.005806 -3.1415926
- joint joint3: limit lower=-2.967 upper=0 effort=100 velocity=5 -> lower=-2.9670597 upper=0 effort=100 velocity=5; origin xyz=0.28503 0 0 rpy=0 0 -1.7939 -> xyz=0.28503 0 0 rpy=0 0 2.8380798
- joint joint4: limit lower=-1.745 upper=1.745 effort=100 velocity=5 -> lower=-1.553343 upper=1.553343 effort=100 velocity=5; origin xyz=-0.021984 -0.25075 0 rpy=1.5708 0 0 -> xyz=0.27364 0 0 rpy=0 0 0.0806342
- joint joint5: limit lower=-1.22 upper=1.22 effort=100 velocity=5 -> lower=-1.553343 upper=1.553343 effort=100 velocity=5; origin xyz=0 0 0 rpy=-1.5708 0 0 -> xyz=0.07466 0 0 rpy=-1.5707963 1.5707963 0
- joint joint6: limit lower=-2.0944 upper=2.0944 effort=100 velocity=3 -> lower=-2.0943951 upper=2.0943951 effort=100 velocity=5; origin xyz=8.8259E-05 -0.091 0 rpy=1.5708 0 0 -> xyz=0 -0.035 0 rpy=1.5707963 0 0
